File: _autosave-altimeter.kicad_pcb (KiCad board)
At the start: 2 copper layers, 45 x 24 mm, 50 parts, among them J201 Conn_01x10, J202 Conn_ARM_JTAG_SWD_10, J203 Conn_02x03_Counter_Clockwise, J204 Conn_01x04, J205 USB_B_Micro, Q101 DMG2301L, Q302 BC847BDW1, Q402 BC847BDW1, Q502 BC847BDW1, U101 STM32F302CCTx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

Commit message: update pyro output stage. add a fuse to the test circuit and remove pullup for sense line
Signed-off-by: Thomas Schmid <tom@binary-kitchen.de>
Parts:
- removed R302, R305, R402, R405, R502, R505: R, Resistor_SMD:R_0402_1005Metric
- R301, R304, R401, R404, R501, R504: value R -> 2.7k
- R303, R403, R503: value R -> 33
Connections:
- Q302 pad 6: Net-(Q302-Pad6) -> PYRO1_LOW
- Q402 pad 6: Net-(Q402-Pad6) -> PYRO2_LOW
- Q502 pad 6: Net-(Q502-Pad6) -> PYRO3_LOW
Routing:
- net PYRO1_LOW: track 0.00 -> 1.16 mm
- net Net-(Q302-Pad6): track 1.16 -> 0.00 mm
