File: altimeter.kicad_pcb (KiCad board)
At the start: 4 copper layers, 45 x 24 mm, 85 parts, among them J201 Conn_01x10, J202 Conn_ARM_JTAG_SWD_10, J203 Conn_02x03_Counter_Clockwise, J204 USB_B_Micro, J205 Conn_01x04, Q1 BC848CDW1T1G, Q101 DMG2301L, Q102 NTR4003NT1G, Q103 SISS05dn, Q301 BC848CDW1T1G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

Commit message: first prototyp order
Signed-off-by: Thomas Schmid <tom@binary-kitchen.de>
Parts:
- added D102: LED, LED_SMD:LED_0603_1608Metric, F.Cu at (162.0, 106.2)
- R105: value 100k -> 680
- moved R105 6.78 mm to (163.6, 103.9)
Connections:
- Q103 pad 4: Net-(D102-Pad1) -> GND
- R105 pad 1: Net-(D102-Pad1) -> Net-(D102-Pad2)
- R105 pad 2: GND -> +3V3
Routing:
- net +3V3: track 53.1 -> 55.6 mm
- net Net-(D102-Pad2): track 0.00 -> 2.25 mm
- net GND: track 127.3 -> 128.6 mm, vias 67 -> 64
Other:
- rule solder_mask_min_width: 0.1 -> 0.0889
- board text added: "+"
- board text added: "-"
- board text added: "Alturia Altimeter CC-BY-NC-SA 4.0 T. Schmid © 2019"
- board text removed: "CC-BY-NC-SA 4.0"

Commit message: fix untinted vias
Signed-off-by: Thomas Schmid <tom@binary-kitchen.de>
Other:
- board text added: "V1.0 rev.B"
Changed lines of the file:
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@@
-(kicad_pcb (version 20171130) (host pcbnew 5.1.4)
+(kicad_pcb (version 20171130) (host pcbnew "(5.1.4)-1")
   (general
     (thickness 1.6)
-    (drawings 28)
+    (drawings 29)
     (tracks 1248)
     (zones 0)
@@
       (usegerberattributes false)
       (usegerberadvancedattributes false)
-      (creategerberjobfile false)
+      (creategerberjobfile true)
       (excludeedgelayer true)
       (linewidth 0.100000)
       (plotframeref false)
-      (viasonmask true)
+      (viasonmask false)
       (mode 1)
       (useauxorigin false)
@@
       (plotinvisibletext false)
       (padsonsilk false)
-      (subtractmaskfromsilk false)
+      (subtractmaskfromsilk true)
       (outputformat 1)
       (mirror false)
@@
     )
   )
+  (gr_text "V1.0 rev.B" (at 165.9 102.2 180) (layer B.SilkS)
+    (effects (font (size 0.762 0.762) (thickness 0.1905)) (justify mirror))
+  )
   (gr_text - (at 174.244 119.634 270) (layer F.SilkS)

Commit message: changed mcu from stm32f302xc to stm32f303xc
Signed-off-by: Thomas Schmid <tom@binary-kitchen.de>
Parts:
- U101: value STM32F302CCTx -> STM32F303CCTx
Connections:
- U101 pad 3: Net-(C101-Pad1) -> Net-(U101-Pad3)
Changed lines of the file:
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@@
     (zones 0)
     (modules 86)
-    (nets 83)
+    (nets 84)
   )
   (page A4)
@@
   (net 81 +BATT)
   (net 82 "Net-(D102-Pad2)")
+  (net 83 "Net-(U101-Pad3)")
   (net_class Default "Dies ist die voreingestellte Netzklasse."
     (clearance 0.1651)
@@
     (add_net "Net-(Q501-Pad2)")
     (add_net "Net-(R103-Pad2)")
+    (add_net "Net-(U101-Pad3)")
     (add_net "Net-(U102-Pad11)")
     (add_net "Net-(U102-Pad12)")
@@
       (effects (font (size 1 1) (thickness 0.15)) (justify mirror))
     )
-    (fp_text value STM32F302CCTx (at 0 -5.85) (layer B.Fab) hide
+    (fp_text value STM32F303CCTx (at 0 -5.85) (layer B.Fab) hide
       (effects (font (size 1 1) (thickness 0.15)) (justify mirror))
     )
@@
       (net 3 "Net-(C102-Pad1)"))
     (pad 3 smd roundrect (at -4.1625 1.75) (size 1.475 0.3) (layers B.Cu B.Paste B.Mask) (roundrect_rratio 0.25)
-      (net 2 "Net-(C101-Pad1)"))
+      (net 83 "Net-(U101-Pad3)"))
     (pad 2 smd roundrect (at -4.1625 2.25) (size 1.475 0.3) (layers B.Cu B.Paste B.Mask) (roundrect_rratio 0.25)
       (net 80 FLASH_HOLD))
