File: altimeter.sch (KiCad schematic (older format))
At the start: 32 parts, among them Q101 DMG2301L, Q102 DMG2301L, U1 LMV331, U101 STM32F302CCTx, U102 MT25Q, U103 AIS2120SXTR, U104 MIC5219-3.3YM5, U105 LF50_TO252, U107 MS5611-01BA, Y1 Crystal_GND24

Commit message: major work on layout. nearly finished
Signed-off-by: Thomas Schmid <tom@binary-kitchen.de>
Parts:
- removed U102: MT25Q, Package_SO:SOIC-16W_7.5x10.3mm_P1.27mm, symbol altimeter:MT25Q
- added C111, C112, C113, C114, C115, C116: C_Small, Capacitor_SMD:C_0402_1005Metric, symbol Device:C_Small
- added U102: S25L512S, Package_SO:SOIC-16W_7.5x10.3mm_P1.27mm, symbol altimeter:S25L512S
- C1, C2: footprint (none) -> Capacitor_SMD:C_0402_1005Metric
- C106: footprint Capacitor_SMD:C_0603_1608Metric_Pad1.05x0.95mm_HandSolder -> Capacitor_SMD:C_0402_1005Metric
- C109, C110: renamed from C?; footprint (none) -> Capacitor_SMD:C_0402_1005Metric
- U1: footprint (none) -> Package_TO_SOT_SMD:SOT-23-5
- gave numbers to parts that had none: 1
Connections:
- net labels added: SWO
- net labels removed: BARO_CSS, JTDO
- wire segments 158 -> 182
Other:
- note removed: "Replace Flash with JEDEC compatible flash for zephyr compatibility"
Changed lines of the file:
@@
 SWDIO
 Text GLabel 1750 2700 0    50   Input ~ 0
-JTDO
+SWO
 Text GLabel 1750 3600 0    50   Input ~ 0
 SPI2_NSS
@@
 	1    0    0    -1
 $EndComp
-Text GLabel 1750 2600 0    50   Input ~ 0
-BARO_CSS
+Text GLabel 1750 2500 0    50   Input ~ 0
+BARO_CS
 Text GLabel 9300 5250 0    50   Input ~ 0
 SPI1_SCK
@@
 F 0 "C106" V 9771 4700 50  0000 C CNN
 F 1 "100n" V 9862 4700 50  0000 C CNN
-F 2 "Capacitor_SMD:C_0603_1608Metric_Pad1.05x0.95mm_HandSolder" H 10000 4700 50  0001 C CNN
+F 2 "Capacitor_SMD:C_0402_1005Metric" H 10000 4700 50  0001 C CNN
 F 3 "~" H 10000 4700 50  0001 C CNN
 	1    10000 4700
@@
 Connection ~ 10750 2350
 $Comp
-L altimeter:MT25Q U102
-U 1 1 5D55332E
-P 6000 4850
-F 0 "U102" H 6228 4246 50  0000 L CNN
-F 1 "MT25Q" H 6228 4155 50  0000 L CNN
-F 2 "Package_SO:SOIC-16W_7.5x10.3mm_P1.27mm" H 7100 4250 50  0001 C CNN
-F 3 "" H 6000 4850 50  0001 C CNN
-	1    6000 4850
-	1    0    0    -1
-$EndComp
-$Comp
 L power:+3.3V #PWR0109
 U 1 1 5D56315F
@@
 Text GLabel 7250 4950 0    50   Input ~ 0
 ACC_CS
-Text GLabel 1750 3400 0    50   Input ~ 0
+Text GLabel 1750 2400 0    50   Input ~ 0
 ACC_CS
 Wire Wire Line
@@
 F 0 "C2" V 8021 4650 50  0000 C CNN
 F 1 "100n" V 8112 4650 50  0000 C CNN
-F 2 "" H 8250 4650 50  0001 C CNN
+F 2 "Capacitor_SMD:C_0402_1005Metric" H 8250 4650 50  0001 C CNN
 F 3 "~" H 8250 4650 50  0001 C CNN
 	1    8250 4650
@@
 F 0 "C1" V 6071 4600 50  0000 C CNN
 F 1 "100n" V 6162 4600 50  0000 C CNN
-F 2 "" H 6300 4600 50  0001 C CNN
+F 2 "Capacitor_SMD:C_0402_1005Metric" H 6300 4600 50  0001 C CNN
 F 3 "~" H 6300 4600 50  0001 C CNN
 	1    6300 4600
@@
 F 0 "U1" H 9944 1446 50  0000 L CNN
 F 1 "LMV331" H 9944 1355 50  0000 L CNN
-F 2 "" H 9600 1500 50  0001 C CNN
+F 2 "Package_TO_SOT_SMD:SOT-23-5" H 9600 1500 50  0001 C CNN
 F 3 "http://www.ti.com/lit/ds/symlink/lmv331.pdf" H 9600 1600 50  0001 C CNN
 	1    9600 1400
@@
 Text GLabel 3050 3400 2    50   Input ~ 0
 UART1_RX
-Text GLabel 1750 3500 0    50   Input ~ 0
+Text GLabel 1750 3400 0    50   Input ~ 0
 IMU_ACC_CS
 Text GLabel 1750 3200 0    50   Input ~ 0
@@
 	1    0    0    -1
 $EndComp
-Text GLabel 1750 2500 0    50   Input ~ 0
+Text GLabel 1750 3500 0    50   Input ~ 0
 SUMMER
 Wire Wire Line
@@
 SPI1_SCK
 $Comp
-L altimeter:BMI088 U?
+L altimeter:BMI088 U106
 U 1 1 5D631374
 P 5800 3600
-F 0 "U?" H 5800 4725 50  0000 C CNN
+F 0 "U106" H 5800 4725 50  0000 C CNN
 F 1 "BMI088" H 5800 4634 50  0000 C CNN
 F 2 "" H 5650 3650 50  0001 C CNN
@@
 $EndComp
 $Comp
-L power:GND #PWR?
+L power:GND #PWR0141
 U 1 1 5D64A47E
 P 5200 3850
-F 0 "#PWR?" H 5200 3600 50  0001 C CNN
+F 0 "#PWR0141" H 5200 3600 50  0001 C CNN
 F 1 "GND" H 5205 3677 50  0000 C CNN
 F 2 "" H 5200 3850 50  0001 C CNN
@@
 Connection ~ 5200 3600
 $Comp
-L power:GND #PWR?
+L power:GND #PWR0142
 U 1 1 5D656842
 P 6400 3850
-F 0 "#PWR?" H 6400 3600 50  0001 C CNN
+F 0 "#PWR0142" H 6400 3600 50  0001 C CNN
 F 1 "GND" H 6405 3677 50  0000 C CNN
 F 2 "" H 6400 3850 50  0001 C CNN
@@
 Wire Wire Line
 	5050 3200 5300 3200
-Text GLabel 1750 2400 0    50   Input ~ 0
+Text GLabel 1750 2600 0    50   Input ~ 0
 IMU_GYRO_CS
 Wire Wire Line
@@
 	1200 2300 1550 2300
 $Comp
-L power:+3.3V #PWR?
+L power:+3.3V #PWR0143
 U 1 1 5D6DDAC8
 P 7000 3100
-F 0 "#PWR?" H 7000 2950 50  0001 C CNN
+F 0 "#PWR0143" H 7000 2950 50  0001 C CNN
 F 1 "+3.3V" H 6900 3250 50  0000 C CNN
 F 2 "" H 7000 3100 50  0001 C CNN
@@
 $EndComp
 $Comp
-L Device:C_Small C?
+L Device:C_Small C109
 U 1 1 5D6E0200
 P 6600 3550
-F 0 "C?" V 6371 3550 50  0000 C CNN
+F 0 "C109" V 6371 3550 50  0000 C CNN
 F 1 "100n" V 6462 3550 50  0000 C CNN
-F 2 "" H 6600 3550 50  0001 C CNN
+F 2 "Capacitor_SMD:C_0402_1005Metric" H 6600 3550 50  0001 C CNN
 F 3 "~" H 6600 3550 50  0001 C CNN
 	1    6600 3550
@@
 $EndComp
 $Comp
-L Device:C_Small C?
+L Device:C_Small C110
 U 1 1 5D704C25
 P 7000 3550
-F 0 "C?" V 6771 3550 50  0000 C CNN
+F 0 "C110" V 6771 3550 50  0000 C CNN
 F 1 "100n" V 6862 3550 50  0000 C CNN
-F 2 "" H 7000 3550 50  0001 C CNN
+F 2 "Capacitor_SMD:C_0402_1005Metric" H 7000 3550 50  0001 C CNN
 F 3 "~" H 7000 3550 50  0001 C CNN
 	1    7000 3550
@@
 Text GLabel 1750 1800 0    50   Input ~ 0
 INT2
-Text Notes 4450 6000 0    50   ~ 0
-Replace Flash with JEDEC compatible flash for zephyr compatibility
+$Comp
+L altimeter:S25L512S U102
+U 1 1 5D50B565
+P 6000 4850
+F 0 "U102" H 6344 4546 50  0000 L CNN
+F 1 "S25L512S" H 6344 4455 50  0000 L CNN
+F 2 "Package_SO:SOIC-16W_7.5x10.3mm_P1.27mm" H 7100 4250 50  0001 C CNN
+F 3 "" H 6000 4850 50  0001 C CNN
+	1    6000 4850
+	1    0    0    -1
+$EndComp
+$Comp
+L Device:C_Small C111
+U 1 1 5D512E0A
+P 3300 950
+F 0 "C111" H 3392 996 50  0000 L CNN
+F 1 "C_Small" H 3392 905 50  0000 L CNN
+F 2 "Capacitor_SMD:C_0402_1005Metric" H 3300 950 50  0001 C CNN
+F 3 "~" H 3300 950 50  0001 C CNN
+	1    3300 950
+	1    0    0    -1
+$EndComp
+$Comp
+L Device:C_Small C113
+U 1 1 5D513394
+P 3500 950
+F 0 "C113" H 3592 996 50  0000 L CNN
+F 1 "C_Small" H 3592 905 50  0000 L CNN
+F 2 "Capacitor_SMD:C_0402_1005Metric" H 3500 950 50  0001 C CNN
+F 3 "~" H 3500 950 50  0001 C CNN
+	1    3500 950
+	1    0    0    -1
+$EndComp
+$Comp
+L Device:C_Small C115
+U 1 1 5D51377B
+P 3700 950
+F 0 "C115" H 3792 996 50  0000 L CNN
+F 1 "C_Small" H 3792 905 50  0000 L CNN
+F 2 "Capacitor_SMD:C_0402_1005Metric" H 3700 950 50  0001 C CNN
+F 3 "~" H 3700 950 50  0001 C CNN
+	1    3700 950
+	1    0    0    -1
+$EndComp
+$Comp
+L Device:C_Small C116
+U 1 1 5D513A48
+P 3900 950
+F 0 "C116" H 3992 996 50  0000 L CNN
+F 1 "C_Small" H 3992 905 50  0000 L CNN
+F 2 "Capacitor_SMD:C_0402_1005Metric" H 3900 950 50  0001 C CNN
+F 3 "~" H 3900 950 50  0001 C CNN
+	1    3900 950
+	1    0    0    -1
+$EndComp
+$Comp
+L Device:C_Small C112
+U 1 1 5D51426E
+P 3300 1950
+F 0 "C112" H 3392 1996 50  0000 L CNN
+F 1 "C_Small" H 3392 1905 50  0000 L CNN
+F 2 "Capacitor_SMD:C_0402_1005Metric" H 3300 1950 50  0001 C CNN
+F 3 "~" H 3300 1950 50  0001 C CNN
+	1    3300 1950
+	1    0    0    -1
+$EndComp
+$Comp
+L Device:C_Small C114
+U 1 1 5D514560
+P 3500 1950
+F 0 "C114" H 3592 1996 50  0000 L CNN
+F 1 "C_Small" H 3592 1905 50  0000 L CNN
+F 2 "Capacitor_SMD:C_0402_1005Metric" H 3500 1950 50  0001 C CNN
+F 3 "~" H 3500 1950 50  0001 C CNN
+	1    3500 1950
+	1    0    0    -1
+$EndComp
+$Comp
+L power:+3.3V #PWR0144
+U 1 1 5D519CA6
+P 3300 650
+F 0 "#PWR0144" H 3300 500 50  0001 C CNN
+F 1 "+3.3V" H 3315 823 50  0000 C CNN
+F 2 "" H 3300 650 50  0001 C CNN
+F 3 "" H 3300 650 50  0001 C CNN
+	1    3300 650
+	1    0    0    -1
+$EndComp
+Wire Wire Line
+	3300 650  3300 750
+Wire Wire Line
+	3300 750  3500 750
+Wire Wire Line
+	3500 750  3500 850
+Connection ~ 3300 750
+Wire Wire Line
+	3300 750  3300 850
+Wire Wire Line
+	3500 750  3700 750
+Wire Wire Line
+	3700 750  3700 850
+Connection ~ 3500 750
+Wire Wire Line
+	3700 750  3900 750
+Wire Wire Line
+	3900 750  3900 850
+Connection ~ 3700 750
+$Comp
+L power:GND #PWR0145
+U 1 1 5D541B40
+P 3300 1200
+F 0 "#PWR0145" H 3300 950 50  0001 C CNN
+F 1 "GND" H 3305 1027 50  0000 C CNN
+F 2 "" H 3300 1200 50  0001 C CNN
+F 3 "" H 3300 1200 50  0001 C CNN
+	1    3300 1200
+	1    0    0    -1
+$EndComp
+Wire Wire Line
+	3300 1200 3300 1150
+Wire Wire Line
+	3300 1150 3500 1150
+Wire Wire Line
+	3500 1150 3500 1050
+Connection ~ 3300 1150
+Wire Wire Line
+	3300 1150 3300 1050
+Wire Wire Line
+	3500 1150 3700 1150
+Wire Wire Line
+	3700 1150 3700 1050
+Connection ~ 3500 1150
+Wire Wire Line
+	3700 1150 3900 1150
+Wire Wire Line
+	3900 1150 3900 1050
+Connection ~ 3700 1150
+$Comp
+L power:+3.3V #PWR0146
+U 1 1 5D56E4D1
+P 3300 1650
+F 0 "#PWR0146" H 3300 1500 50  0001 C CNN
+F 1 "+3.3V" H 3315 1823 50  0000 C CNN
+F 2 "" H 3300 1650 50  0001 C CNN
+F 3 "" H 3300 1650 50  0001 C CNN
+	1    3300 1650
+	1    0    0    -1
+$EndComp
+Wire Wire Line
+	3300 1850 3300 1750
+Wire Wire Line
+	3300 1750 3500 1750
+Wire Wire Line
+	3500 1750 3500 1850
+Connection ~ 3300 1750
+Wire Wire Line
+	3300 1750 3300 1650
+$Comp
+L power:GND #PWR0147
+U 1 1 5D5858EC
+P 3300 2200
+F 0 "#PWR0147" H 3300 1950 50  0001 C CNN
+F 1 "GND" H 3305 2027 50  0000 C CNN
+F 2 "" H 3300 2200 50  0001 C CNN
+F 3 "" H 3300 2200 50  0001 C CNN
+	1    3300 2200
+	1    0    0    -1
+$EndComp
+Wire Wire Line
+	3300 2200 3300 2150
+Wire Wire Line
+	3300 2150 3500 2150
+Wire Wire Line
+	3500 2150 3500 2050
+Connection ~ 3300 2150
+Wire Wire Line
+	3300 2150 3300 2050
 $EndSCHEMATC

Commit message: nearly finished with lacout. Added logo
Signed-off-by: Thomas Schmid <tom@binary-kitchen.de>
Parts:
- added R102: 2.7k, Resistor_SMD:R_0402_1005Metric, symbol Device:R
- C1, C106, C109, C110, C2: Mouser_Link (none) -> https://www.mouser.de/ProductDetail/Wurth-Elektronik/885012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; Parnumber (none) -> 885012205037
- C101, C102: Mouser_Link (none) -> https://www.mouser.de/ProductDetail/Murata-Electronics/GCM1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; Parnumber (none) -> GCM1555G1H220JA16D
- C103: Mouser_Link (none) -> https://www.mouser.de/ProductDetail/Yageo/CC0603KRX5R8BB105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; Parnumber (none) -> CC0603KRX5R8BB105
- C104: Mouser_Link (none) -> https://www.mouser.de/ProductDetail/KEMET/C0805C104Z3VACTU?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; Parnumber (none) -> C0805C104Z3VACTU
- C105: value C_Small -> 470p; Mouser_Link (none) -> https://www.mouser.de/ProductDetail/Taiyo-Yuden/TMK063CG471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; Parnumber (none) -> TMK063CG471JT-F
- C107: Mouser_Link (none) -> https://www.mouser.de/ProductDetail/Taiyo-Yuden/EMK107BJ225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; Parnumber (none) -> EMK107BJ225MA-T
- C108: value C_Small -> 4.7u; Mouser_Link (none) -> https://www.mouser.de/ProductDetail/Taiyo-Yuden/EMK107ABJ47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; Parnumber (none) -> EMK107ABJ475KA-T
- C111, C112, C113, C114, C115, C116: value C_Small -> 100n; Mouser_Link (none) -> https://www.mouser.de/ProductDetail/Wurth-Elektronik/885012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; Parnumber (none) -> 885012205037
- C3: Mouser_Link (none) -> https://www.mouser.de/ProductDetail/Illinois-Capacitor-CDE/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; Parnumber (none) -> 337TTA016M
- D101: Mouser_Link (none) -> https://www.mouser.de/ProductDetail/Kingbright/APTD1608LSUR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; Parnumber (none) -> APTD1608LSURCK
- D103: Mouser_Link (none) -> https://www.mouser.de/ProductDetail/ON-Semiconductor-Fairch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; Parnumber (none) -> 1N4148WS
- LS101: Mouser_Link (none) -> https://www.mouser.de/ProductDetail/CUI/CSS-95B30-SMT-TR?qs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; Parnumber (none) -> CSS-95B30-SMT-TR
- Q101: symbol Device:Q_PMOS_DGS -> Device:Q_PMOS_GSD; Mouser_Link (none) -> https://www.mouser.de/ProductDetail/Diodes-Incorporated/DMG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; Parnumber (none) -> DMG2301L-7
- Q102: value DMG2301L -> NTR4003NT1G; symbol Device:Q_PMOS_DGS -> Device:Q_NMOS_GSD; Mouser_Link (none) -> https://www.mouser.de/ProductDetail/ON-Semiconductor/NTR400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; Parnumber (none) -> NTR4003NT1G
- R1: Mouser_Link (none) -> https://www.mouser.de/ProductDetail/Vishay-Dale/CRCW0402768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; Parnumber (none) -> CRCW040268K0FKEDC
- R101: Mouser_Link (none) -> https://www.mouser.de/ProductDetail/Vishay-Dale/CRCW0402680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; Parnumber (none) -> CRCW0402680RFKEDC
- R103, R104: Mouser_Link (none) -> https://www.mouser.de/ProductDetail/Vishay-Dale/CRCW0402100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; Parnumber (none) -> CRCW0402100KFKEDC
- R2: Mouser_Link (none) -> https://www.mouser.de/ProductDetail/Vishay-Dale/CRCW0402220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; Parnumber (none) -> CRCW0402220KFKEDC
- U1: Mouser_Link (none) -> https://www.mouser.de/ProductDetail/ON-Semiconductor/LMV331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; Parnumber (none) -> LMV331SN3T1G
- U101: Mouser_Link (none) -> https://www.mouser.de/ProductDetail/STMicroelectronics/STM3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; Parnumber (none) -> STM32F302CCT6
- U102: value S25L512S -> S25FL512SAGMFIR11; Mouser_Link (none) -> https://www.mouser.de/ProductDetail/Cypress-Semiconductor/S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; Parnumber (none) -> S25FL512SAGMFIR11
- U103: Mouser_Link (none) -> https://www.mouser.de/ProductDetail/STMicroelectronics/AIS2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; Parnumber (none) -> AIS2120SXTR
- U104: Mouser_Link (none) -> https://www.mouser.de/ProductDetail/Microchip-Technology-Mi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; Parnumber (none) -> MIC5219-3.3YM5-TR
- U105: Mouser_Link (none) -> https://www.mouser.de/ProductDetail/STMicroelectronics/LF50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; Parnumber (none) -> LF50ABDT-TR
- U106: footprint (none) -> altimeter:BMI088; Mouser_Link (none) -> https://www.mouser.de/ProductDetail/Bosch-Sensortec/BMI088?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; Parnumber (none) -> BMI088
- U107: Mouser_Link (none) -> https://www.mouser.de/ProductDetail/Measurement-Specialties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; Parnumber (none) -> MS560702BA03-50
Connections:
- wire segments 182 -> 184
- no-connect marks 2 -> 3
Other:
- note added: "ToDo's:\n\n- USB Schutzdioden\n- ESD Schutzkondensatoren"

Commit message: completed layout
Signed-off-by: Thomas Schmid <tom@binary-kitchen.de>
Parts:
- added D102: D_Zener, symbol Device:D_Zener
- added Q103: SI7149ADP, Package_SO:PowerPAK_SO-8_Single, symbol altimeter:SI7149ADP
- added R105: R, symbol Device:R
Connections:
- net +3V3: no longer U102.1 (HOLD#/IO3)
- net +BATT: now also Q103.5 (D)
- net GND: now also R105.2
- net FLASH_HOLD: now reaches U101.2 (PC13)
- net FLASH_HOLD: now also U102.1 (HOLD#/IO3)
- new net: D102.1 (K), Q103.4 (G), R105.1
- new net VPP: D102.2 (A), Q103.1 (S), Q103.2 (S), Q103.3 (S)
- no-connect marks 3 -> 2
Changed lines of the file:
@@
 	2250 1000 2250 1100
 $Sheet
-S 4850 6550 1550 750
+S 4250 6800 1550 750
 U 5D3DE309
 F0 "Connectors" 50
@@
 F 3 "" H 5300 5400 50  0001 C CNN
 	1    5300 5400
-	0    -1   -1   0
-$EndComp
-$Comp
-L power:+3.3V #PWR0108
-U 1 1 5D5786CD
-P 5300 5500
-F 0 "#PWR0108" H 5300 5350 50  0001 C CNN
-F 1 "+3.3V" V 5315 5628 50  0000 L CNN
-F 2 "" H 5300 5500 50  0001 C CNN
-F 3 "" H 5300 5500 50  0001 C CNN
-	1    5300 5500
 	0    -1   -1   0
 $EndComp
@@
 	1    0    0    -1
 $EndComp
-NoConn ~ 1750 2000
 $Comp
 L power:PWR_FLAG #FLG0102
@@
 Text Notes 11800 700  0    50   ~ 0
 ToDo's:\n\n- USB Schutzdioden\n- ESD Schutzkondensatoren
+Text GLabel 5300 5500 0    50   Input ~ 0
+FLASH_HOLD
+Text GLabel 1250 1500 0    50   Input ~ 0
+FLASH_HOLD
+Wire Wire Line
+	1750 2000 1600 2000
+Wire Wire Line
+	1600 2000 1600 1850
+Wire Wire Line
+	1600 1850 1400 1850
+Wire Wire Line
+	1400 1850 1400 1500
+Wire Wire Line
+	1400 1500 1250 1500
+$Comp
+L power:+BATT #PWR0162
+U 1 1 5D71F539
+P 6550 1650
+F 0 "#PWR0162" H 6550 1500 50  0001 C CNN
+F 1 "+BATT" H 6565 1823 50  0000 C CNN
+F 2 "" H 6550 1650 50  0001 C CNN
+F 3 "" H 6550 1650 50  0001 C CNN
+	1    6550 1650
+	1    0    0    -1
+$EndComp
+Wire Wire Line
+	6550 1650 6550 1700
+Wire Wire Line
+	6550 1700 6850 1700
+$Comp
+L power:VPP #PWR0163
+U 1 1 5D72B18F
+P 7550 1650
+F 0 "#PWR0163" H 7550 1500 50  0001 C CNN
+F 1 "VPP" H 7565 1823 50  0000 C CNN
+F 2 "" H 7550 1650 50  0001 C CNN
+F 3 "" H 7550 1650 50  0001 C CNN
+	1    7550 1650
+	1    0    0    -1
+$EndComp
+Wire Wire Line
+	7550 1650 7550 1700
+Wire Wire Line
+	7550 1700 7400 1700
+$Comp
+L power:GND #PWR0164
+U 1 1 5D749A10
+P 7050 2550
+F 0 "#PWR0164" H 7050 2300 50  0001 C CNN
+F 1 "GND" H 7055 2377 50  0000 C CNN
+F 2 "" H 7050 2550 50  0001 C CNN
+F 3 "" H 7050 2550 50  0001 C CNN
+	1    7050 2550
+	1    0    0    -1
+$EndComp
+$Comp
+L Device:D_Zener D102
+U 1 1 5D74B84D
+P 7400 1900
+F 0 "D102" V 7446 1821 50  0000 R CNN
+F 1 "D_Zener" V 7355 1821 50  0000 R CNN
+F 2 "" H 7400 1900 50  0001 C CNN
+F 3 "~" H 7400 1900 50  0001 C CNN
+	1    7400 1900
+	0    -1   -1   0
+$EndComp
+$Comp
+L Device:R R105
+U 1 1 5D74CCF3
+P 7050 2300
+F 0 "R105" H 7120 2346 50  0000 L CNN
+F 1 "R" H 7120 2255 50  0000 L CNN
+F 2 "" V 6980 2300 50  0001 C CNN
+F 3 "~" H 7050 2300 50  0001 C CNN
+	1    7050 2300
+	1    0    0    -1
+$EndComp
+Wire Wire Line
+	7050 2000 7050 2100
+Wire Wire Line
+	7050 2100 7400 2100
+Wire Wire Line
+	7400 2100 7400 2050
+Wire Wire Line
+	7400 1750 7400 1700
+Connection ~ 7400 1700
+Wire Wire Line
+	7400 1700 7250 1700
+Wire Wire Line
+	7050 2550 7050 2450
+Wire Wire Line
+	7050 2150 7050 2100
+Connection ~ 7050 2100
+$Comp
+L altimeter:SI7149ADP Q103
+U 1 1 5D7A8BFD
+P 7050 1800
+F 0 "Q103" V 7393 1800 50  0000 C CNN
+F 1 "SI7149ADP" V 7302 1800 50  0000 C CNN
+F 2 "Package_SO:PowerPAK_SO-8_Single" H 7250 1900 50  0001 C CNN
+F 3 "~" H 7050 1800 50  0001 C CNN
+	1    7050 1800
+	0    -1   -1   0
+$EndComp
 $EndSCHEMATC

Commit message: minor updates
Signed-off-by: Thomas Schmid <tom@lfence.de>
Parts:
- Q103: value SI7149ADP -> SISS05dn; footprint Package_SO:PowerPAK_SO-8_Single -> Package_SO:Vishay_PowerPAK_1212-8_Single
- R105: value R -> 100k; footprint (none) -> Resistor_SMD:R_0402_1005Metric; Mouser_Link (none) -> https://www.mouser.de/ProductDetail/Vishay-Dale/CRCW0402100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; Parnumber (none) -> CRCW0402100KFKEDC
Connections:
- net +BATT: no longer C104.1, C3.1, R103.1, R2.2, U105.1 (VI)
- net VPP: now also C104.1, C3.1, R103.1, R2.2, U105.1 (VI)
Other:
- note removed: "ToDo's:\n\n- USB Schutzdioden\n- ESD Schutzkondensatoren"
Changed lines of the file:
@@
 	9900 1400 10100 1400
-$Comp
-L power:+BATT #PWR0113
-U 1 1 5D4664F5
-P 8750 1000
-F 0 "#PWR0113" H 8750 850 50  0001 C CNN
-F 1 "+BATT" H 8765 1173 50  0000 C CNN
-F 2 "" H 8750 1000 50  0001 C CNN
-F 3 "" H 8750 1000 50  0001 C CNN
-	1    8750 1000
-	1    0    0    -1
-$EndComp
 $Comp
 L Device:R_Small R104
@@
 Wire Wire Line
 	9350 3450 9350 3550
-$Comp
-L power:+BATT #PWR0115
-U 1 1 5D4E69FF
-P 9350 3300
-F 0 "#PWR0115" H 9350 3150 50  0001 C CNN
-F 1 "+BATT" H 9365 3473 50  0000 C CNN
-F 2 "" H 9350 3300 50  0001 C CNN
-F 3 "" H 9350 3300 50  0001 C CNN
-	1    9350 3300
-	1    0    0    -1
-$EndComp
 Wire Wire Line
 	9350 3300 9350 3450
@@
 Wire Wire Line
 	2000 5150 2000 5400
-$Comp
-L power:+BATT #PWR0132
-U 1 1 5D50022D
-P 2000 5150
-F 0 "#PWR0132" H 2000 5000 50  0001 C CNN
-F 1 "+BATT" H 2015 5323 50  0000 C CNN
-F 2 "" H 2000 5150 50  0001 C CNN
-F 3 "" H 2000 5150 50  0001 C CNN
-	1    2000 5150
-	1    0    0    -1
-$EndComp
 Text GLabel 3050 3300 2    50   Input ~ 0
 UART1_TX
@@
 $EndComp
 Connection ~ 6600 3300
-Text Notes 11800 700  0    50   ~ 0
-ToDo's:\n\n- USB Schutzdioden\n- ESD Schutzkondensatoren
 Text GLabel 5300 5500 0    50   Input ~ 0
 FLASH_HOLD
@@
 P 7050 2300
 F 0 "R105" H 7120 2346 50  0000 L CNN
-F 1 "R" H 7120 2255 50  0000 L CNN
-F 2 "" V 6980 2300 50  0001 C CNN
+F 1 "100k" H 7120 2255 50  0000 L CNN
+F 2 "Resistor_SMD:R_0402_1005Metric" V 6980 2300 50  0001 C CNN
 F 3 "~" H 7050 2300 50  0001 C CNN
+F 4 "https://www.mouser.de/ProductDetail/Vishay-Dale/CRCW0402100KFKED?qs=sGAEpiMZZMu61qfTUdNhG2DpbjADlD3GqPf2An0kBCw%3D" H 7050 2300 50  0001 C CNN "Mouser_Link"
+F 5 "CRCW0402100KFKEDC" H 7050 2300 50  0001 C CNN "Parnumber"
 	1    7050 2300
 	1    0    0    -1
@@
 P 7050 1800
 F 0 "Q103" V 7393 1800 50  0000 C CNN
-F 1 "SI7149ADP" V 7302 1800 50  0000 C CNN
-F 2 "Package_SO:PowerPAK_SO-8_Single" H 7250 1900 50  0001 C CNN
-F 3 "~" H 7050 1800 50  0001 C CNN
+F 1 "SISS05dn" V 7302 1800 50  0000 C CNN
+F 2 "Package_SO:Vishay_PowerPAK_1212-8_Single" H 7250 1900 50  0001 C CNN
+F 3 "https://www.mouser.de/datasheet/2/427/siss05dn-1595673.pdf" H 7050 1800 50  0001 C CNN
 	1    7050 1800
 	0    -1   -1   0
 $EndComp
+$Comp
+L power:VPP #PWR?
+U 1 1 5D715463
+P 2000 5150
+F 0 "#PWR?" H 2000 5000 50  0001 C CNN
+F 1 "VPP" H 2015 5323 50  0000 C CNN
+F 2 "" H 2000 5150 50  0001 C CNN
+F 3 "" H 2000 5150 50  0001 C CNN
+	1    2000 5150
+	1    0    0    -1
+$EndComp
+$Comp
+L power:VPP #PWR?
+U 1 1 5D715F7E
+P 9350 3300
+F 0 "#PWR?" H 9350 3150 50  0001 C CNN
+F 1 "VPP" H 9365 3473 50  0000 C CNN
+F 2 "" H 9350 3300 50  0001 C CNN
+F 3 "" H 9350 3300 50  0001 C CNN
+	1    9350 3300
+	1    0    0    -1
+$EndComp
+$Comp
+L power:VPP #PWR?
+U 1 1 5D7169CC
+P 8750 1000
+F 0 "#PWR?" H 8750 850 50  0001 C CNN
+F 1 "VPP" H 8765 1173 50  0000 C CNN
+F 2 "" H 8750 1000 50  0001 C CNN
+F 3 "" H 8750 1000 50  0001 C CNN
+	1    8750 1000
+	1    0    0    -1
+$EndComp
 $EndSCHEMATC
