File: pyro_outputstage.sch (KiCad schematic (older format))
At the start: 8 parts, among them Q301 BC848CDW1T1G, U301 SI7232DN

Commit message: v1.2 rev A
Signed-off-by: Thomas Schmid <tom@binary-kitchen.de>
Connections:
- net FIRE: now also U301.2 (G); no longer U301.4 (G)
- net GND: now also U301.1 (S); no longer U301.3 (S)
- net PYRO_LOW: now also U301.6 (D); no longer U301.5 (D)
Changed lines of the file:
@@
 Title ""
 Date ""
-Rev ""
+Rev "v 1.2 rev.A"
 Comp ""
 Comment1 ""
@@
 AR Path="/5D48B429/5D4757F5" Ref="R502"  Part="1"
 AR Path="/5D4E7D5B/5D4757F5" Ref="R12"  Part="1"
-F 0 "R302" H 5920 4396 50  0000 L CNN
+F 0 "R12" H 5920 4396 50  0000 L CNN
 F 1 "33" H 5920 4305 50  0000 L CNN
 F 2 "Resistor_SMD:R_0402_1005Metric" V 5780 4350 50  0001 C CNN
@@
 AR Path="/5D48B429/5D47580C" Ref="R503"  Part="1"
 AR Path="/5D4E7D5B/5D47580C" Ref="R13"  Part="1"
-F 0 "R303" V 6293 3500 50  0000 C CNN
+F 0 "R13" V 6293 3500 50  0000 C CNN
 F 1 "2.7k" V 6384 3500 50  0000 C CNN
 F 2 "Resistor_SMD:R_0402_1005Metric" V 6430 3500 50  0001 C CNN
@@
 AR Path="/5D48B429/5D475828" Ref="R501"  Part="1"
 AR Path="/5D4E7D5B/5D475828" Ref="R10"  Part="1"
-F 0 "R301" H 4720 4446 50  0000 L CNN
+F 0 "R10" H 4720 4446 50  0000 L CNN
 F 1 "2.7k" H 4720 4355 50  0000 L CNN
 F 2 "Resistor_SMD:R_0402_1005Metric" V 4580 4400 50  0001 C CNN
@@
 AR Path="/5D48B429/5D475835" Ref="Q501"  Part="1"
 AR Path="/5D4E7D5B/5D475835" Ref="Q1"  Part="1"
-F 0 "Q301" H 6141 3546 50  0000 L CNN
+F 0 "Q1" H 6141 3546 50  0000 L CNN
 F 1 "BC848CDW1T1G" H 6141 3455 50  0000 L CNN
 F 2 "Package_TO_SOT_SMD:SOT-363_SC-70-6" H 6150 3600 50  0001 C CNN
@@
 AR Path="/5D48B429/5D47583B" Ref="Q501"  Part="2"
 AR Path="/5D4E7D5B/5D47583B" Ref="Q1"  Part="2"
-F 0 "Q301" H 6390 4096 50  0000 L CNN
+F 0 "Q1" H 6390 4096 50  0000 L CNN
 F 1 "BC848CDW1T1G" H 6390 4005 50  0000 L CNN
 F 2 "Package_TO_SOT_SMD:SOT-363_SC-70-6" H 6400 4150 50  0001 C CNN
@@
 $Comp
 L altimeter:SI7232DN U301
-U 2 1 5D4F79DE
+U 1 1 5D4F79DE
 P 5150 4050
 AR Path="/5D473C9B/5D4F79DE" Ref="U301"  Part="2"
@@
 AR Path="/5D4E7D5B/5D4F79DE" Ref="U501"  Part="1"
 AR Path="/5D4F79DE" Ref="U501"  Part="1"
-F 0 "U301" H 5256 4096 50  0000 L CNN
+F 0 "U501" H 5256 4096 50  0000 L CNN
 F 1 "SI7232DN" H 5256 4005 50  0000 L CNN
 F 2 "Package_SO:Vishay_PowerPAK_1212-8_Dual" H 5150 4050 50  0001 C CNN
@@
 F 4 "https://www.mouser.de/ProductDetail/Vishay-Siliconix/SI7232DN-T1-GE3?qs=%2Fha2pyFaduiZCEC0X5XOlemXjOWX3oZDDwY4%252BOM6S%252B4%3D" H 5150 4050 50  0001 C CNN "Mouser_Link"
 F 5 "SI7232DN-T1-GE3 " H 5150 4050 50  0001 C CNN "Parnumber"
-	2    5150 4050
+	1    5150 4050
 	1    0    0    -1
 $EndComp
@@
 AR Path="/5D48B429/5D6F3FF8" Ref="F501"  Part="1"
 AR Path="/5D4E7D5B/5D6F3FF8" Ref="F1"  Part="1"
-F 0 "F301" H 5938 2946 50  0000 L CNN
+F 0 "F1" H 5938 2946 50  0000 L CNN
 F 1 "Polyfuse" H 5938 2855 50  0000 L CNN
 F 2 "Fuse:Fuse_0603_1608Metric_Pad1.05x0.95mm_HandSolder" H 5900 2700 50  0001 L CNN
@@
 AR Path="/5D48B429/5D4D8D4C" Ref="R7"  Part="1"
 AR Path="/5D4E7D5B/5D4D8D4C" Ref="R9"  Part="1"
-F 0 "R3" H 4620 2896 50  0000 L CNN
+F 0 "R9" H 4620 2896 50  0000 L CNN
 F 1 "68k" H 4620 2805 50  0000 L CNN
 F 2 "Resistor_SMD:R_0402_1005Metric" V 4480 2850 50  0001 C CNN
@@
 AR Path="/5D48B429/5D4D933B" Ref="R8"  Part="1"
 AR Path="/5D4E7D5B/5D4D933B" Ref="R11"  Part="1"
-F 0 "R4" H 4920 2596 50  0000 L CNN
+F 0 "R11" H 4920 2596 50  0000 L CNN
 F 1 "220k" H 4920 2505 50  0000 L CNN
 F 2 "Resistor_SMD:R_0402_1005Metric" V 4780 2550 50  0001 C CNN

Commit message: update
Signed-off-by: Thomas Schmid <tom@binary-kitchen.de>
Connections:
- net FIRE: now also U301.4 (G); no longer U301.2 (G)
- net GND: now also U301.3 (S); no longer U301.1 (S)
- net PYRO_LOW: now also U301.5 (D); no longer U301.6 (D)
Changed lines of the file:
@@
 $Descr A4 11693 8268
 encoding utf-8
-Sheet 3 6
+Sheet 5 6
 Title ""
 Date ""
@@
 AR Path="/5D48B429/5D4757F5" Ref="R502"  Part="1"
 AR Path="/5D4E7D5B/5D4757F5" Ref="R12"  Part="1"
-F 0 "R12" H 5920 4396 50  0000 L CNN
+F 0 "R502" H 5920 4396 50  0000 L CNN
 F 1 "33" H 5920 4305 50  0000 L CNN
 F 2 "Resistor_SMD:R_0402_1005Metric" V 5780 4350 50  0001 C CNN
@@
 AR Path="/5D48B429/5D47580C" Ref="R503"  Part="1"
 AR Path="/5D4E7D5B/5D47580C" Ref="R13"  Part="1"
-F 0 "R13" V 6293 3500 50  0000 C CNN
+F 0 "R503" V 6293 3500 50  0000 C CNN
 F 1 "2.7k" V 6384 3500 50  0000 C CNN
 F 2 "Resistor_SMD:R_0402_1005Metric" V 6430 3500 50  0001 C CNN
@@
 AR Path="/5D48B429/5D475828" Ref="R501"  Part="1"
 AR Path="/5D4E7D5B/5D475828" Ref="R10"  Part="1"
-F 0 "R10" H 4720 4446 50  0000 L CNN
+F 0 "R501" H 4720 4446 50  0000 L CNN
 F 1 "2.7k" H 4720 4355 50  0000 L CNN
 F 2 "Resistor_SMD:R_0402_1005Metric" V 4580 4400 50  0001 C CNN
@@
 AR Path="/5D48B429/5D475835" Ref="Q501"  Part="1"
 AR Path="/5D4E7D5B/5D475835" Ref="Q1"  Part="1"
-F 0 "Q1" H 6141 3546 50  0000 L CNN
+F 0 "Q501" H 6141 3546 50  0000 L CNN
 F 1 "BC848CDW1T1G" H 6141 3455 50  0000 L CNN
 F 2 "Package_TO_SOT_SMD:SOT-363_SC-70-6" H 6150 3600 50  0001 C CNN
@@
 AR Path="/5D48B429/5D47583B" Ref="Q501"  Part="2"
 AR Path="/5D4E7D5B/5D47583B" Ref="Q1"  Part="2"
-F 0 "Q1" H 6390 4096 50  0000 L CNN
+F 0 "Q501" H 6390 4096 50  0000 L CNN
 F 1 "BC848CDW1T1G" H 6390 4005 50  0000 L CNN
 F 2 "Package_TO_SOT_SMD:SOT-363_SC-70-6" H 6400 4150 50  0001 C CNN
@@
 $Comp
 L altimeter:SI7232DN U301
-U 1 1 5D4F79DE
+U 2 1 5D4F79DE
 P 5150 4050
 AR Path="/5D473C9B/5D4F79DE" Ref="U301"  Part="2"
@@
 F 4 "https://www.mouser.de/ProductDetail/Vishay-Siliconix/SI7232DN-T1-GE3?qs=%2Fha2pyFaduiZCEC0X5XOlemXjOWX3oZDDwY4%252BOM6S%252B4%3D" H 5150 4050 50  0001 C CNN "Mouser_Link"
 F 5 "SI7232DN-T1-GE3 " H 5150 4050 50  0001 C CNN "Parnumber"
-	1    5150 4050
+	2    5150 4050
 	1    0    0    -1
 $EndComp
@@
 AR Path="/5D48B429/5D6F3FF8" Ref="F501"  Part="1"
 AR Path="/5D4E7D5B/5D6F3FF8" Ref="F1"  Part="1"
-F 0 "F1" H 5938 2946 50  0000 L CNN
+F 0 "F501" H 5938 2946 50  0000 L CNN
 F 1 "Polyfuse" H 5938 2855 50  0000 L CNN
 F 2 "Fuse:Fuse_0603_1608Metric_Pad1.05x0.95mm_HandSolder" H 5900 2700 50  0001 L CNN
@@
 AR Path="/5D48B429/5D4D8D4C" Ref="R7"  Part="1"
 AR Path="/5D4E7D5B/5D4D8D4C" Ref="R9"  Part="1"
-F 0 "R9" H 4620 2896 50  0000 L CNN
+F 0 "R7" H 4620 2896 50  0000 L CNN
 F 1 "68k" H 4620 2805 50  0000 L CNN
 F 2 "Resistor_SMD:R_0402_1005Metric" V 4480 2850 50  0001 C CNN
@@
 AR Path="/5D48B429/5D4D933B" Ref="R8"  Part="1"
 AR Path="/5D4E7D5B/5D4D933B" Ref="R11"  Part="1"
-F 0 "R11" H 4920 2596 50  0000 L CNN
+F 0 "R8" H 4920 2596 50  0000 L CNN
 F 1 "220k" H 4920 2505 50  0000 L CNN
 F 2 "Resistor_SMD:R_0402_1005Metric" V 4780 2550 50  0001 C CNN
